File: PCB/synth-zodiac-scorpio-kbd.sch (EAGLE design)
At the start: 59 parts, among them Q1 PMP4201, U3 LM393, U4 TL074A, U5 CD4066

Commit message: Snapshot of designs so far.
Parts:
- removed BIAS: NP, rlc:TRIMPOTTC33X
- removed C1: 4700pF, rlc:CAPACITOR0603
- removed C10: 220pF, rlc:CAPACITOR0603
- removed C3, C4, C6, C7: 0.1uF, rlc:CAPACITOR0603
- removed C5: 3900pF, rlc:CAPACITOR0603
- removed C8: 1.0uF, rlc:CAPACITOR0603
- removed C9: 100pF, rlc:CAPACITOR0603
- removed CONST1: Aquarius, circuit-monkey-zodiac:CONSTELLATION-AQUARIUS
- removed CP_EXP_VCO, CP_VCO_LIN_FM, CP_VCO_OUT: PADSMD-070X070, con-testpoints:PADSMD-070X070
- removed D1, D2: 1N4148, diodes:DIODE-1N4148
- removed EXP_VCO_TRIM: 100K - NP, rlc:TRIMPOTTC33X
- removed FREQ: 10K, rlc:TRIMPOT9MM_PCB_SHAFT
- removed J1: (no value), con-jst:04P-VT-SMT
- removed KB_TRIM: 100K, rlc:TRIMPOTTC33X
- removed PULSE, SAW, TP4: TPSMD-040-RND, con-testpoints:TPSMD-040-RND
- removed PWM_CV, VCO_MOD_CV, VCO_OUT: 2-pin, VT, SMT, con-jst:02PVT-SMT
- removed Q1: PMP4201, transistor-bjt:NPN-DUALPMP4201
- removed R10, R11, R13, R14, R24: 0, rlc:RESISTOR0603
- removed R12: NS, rlc:RESISTOR0603
- removed R15, R16: 100K, rlc:RESISTOR0603
- removed R17: 10.0K, rlc:RESISTOR0603
- removed R18: 4.75M, rlc:RESISTOR0603
- removed R19, R20, R21, R22: 4.99K, rlc:RESISTOR0603
- removed R2, R3: 221K, rlc:RESISTOR0603
- removed R23, R9: 10K, rlc:RESISTOR0603
- removed R4: 412K, rlc:RESISTOR0603
- removed R5: 68.1K - NP, rlc:RESISTOR0603
- removed R6: 2.2K, rlc:RESISTOR0603
- removed R7: 499K, rlc:RESISTOR0603
- removed R8: 1.82M, rlc:RESISTOR0603
- removed TYPE: SPDT, switch-thd:SLIDE-SPDTSS-12-F45-TH-PCB
- removed U3: LM393, op-amp:DUAL-LM393ED
- removed U4: TL074A, op-amp:QUADTL074A-SOIC
- removed U5: CD4066, logic:CD4066SO14
- added A, A#, B, C, C#, D, D#, E, F, F#, G, G#: Tact. Sw., switch-smd:PUSHBTN-MOMB3FS
- added C43, C44, C48, C51, C52, C53, C54, C59: 0.1uF, rlc:CAPACITOR0603
- added C45: 100pF, rlc:CAPACITOR0603
- added C46: 1000pF, rlc:CAPACITOR0603
- added C47: 220pF, rlc:CAPACITOR0603
- added C49: 47pF, rlc:CAPACITOR0603
- added C50: 1.0uF, rlc:CAPACITOR0603
- added CONST: Scorpio, circuit-monkey-zodiac:CONSTELLATION-SCORPIO
- added CP_KB_CV: PAD-70X70SMD-070X070, con-testpoints:PAD-70X70SMD-070X070
- added D10, D11, D12, D13, D14, D15, D16, D17, D18, D19, D20, D5, D6, D7, D8, D9: 1N4148, diodes:DIODE-1N4148
- added GATE, TRIG: 2-pin, VT, SMT, con-jst:02PVT-SMT
- added GLIDE: 1M, rlc:TRIMPOT9MM_PCB_SHAFT
- added PWR: (no value), con-jst:04P-VT-SMT
- added R57, R76: 1.00K, rlc:RESISTOR0603
- added R74: 10.0M, rlc:RESISTOR0603
- added R75: 100K, rlc:RESISTOR0603
- added R77: 4.99K, rlc:RESISTOR0603
- added R78: 47.5K, rlc:RESISTOR0603
- added R79: 10.0K, rlc:RESISTOR0603
- added R80, R81, R82, R83, R84: 1.0M, rlc:RESISTOR0603
- added R85, R86, R87: 499K, rlc:RESISTOR0603
- added U1: 74VHC1G125, logic:74VHC1G125CMOS-SOT553
- added U13: TL072A, op-amp:DUALTL072A
- added U14: CD40106, logic:CD40106-SOP14
- added U15: 40175, logic:CD40175SMT-D-TYPE
- added U16, U19: CD4051, logic:CD4051SO-D
- added U18: CD4520, logic:CD4520
- C2: value 22uF -> Tact. Sw.; device rlc:CAPACITOR0603 -> switch-smd:PUSHBTN-MOMB3FS
- CP_GND: value PADSMD-070X070 -> PAD-70X70SMD-070X070; device con-testpoints:PADSMD-070X070 -> con-testpoints:PAD-70X70SMD-070X070
- GLYPH: value Aquarius -> Scorpio; device circuit-monkey-zodiac:GLYPH-AQUARIUS -> circuit-monkey-zodiac:GLYPH-SCORPIO
Connections:
- removed net BIAS: BIAS.2, R19.2, R20.1, R21.1
- removed net EXP_VCO_CV_IN: CP_EXP_VCO.PAD, EXP_VCO_TRIM.1
- removed net EXP_VCO_LIN_FM: CP_VCO_LIN_FM.PAD, R7.1
- removed net FREQ: FREQ.2, R2.1
- removed net FREQ_CV_MIX: C1.1, R2.2, R3.2, R4.2, R5.2, R6.1, U4-A.-
- removed net N$12: Q1-A.EMITTER, R7.2, R8.2, U4-B.+
- removed net N$13: Q1-B.EMITTER, U4-B.-, U4-B.OUT
- removed net N$14: C1.2, Q1-A.BASE, R6.2, U4-A.OUT
- removed net N$15: R12.2, R9.2, U5-A.EN, U5-B.EN, U5-C.IN
- removed net N$16: C9.1, R17.1, R18.1, U4-D.+
- removed net N$17: R14.2, U3-B.-
- removed net N$18: C9.2, D1.A, R18.2, U4-D.OUT
- removed net N$20: C5.2, Q1-B.COLLECTOR, U4-C.+, U5-A.OUT
- removed net N$21: BIAS.3, C8.2, R17.2, R19.1
- removed net N$22: C10.1, R21.2, U5-B.IN
- removed net N$23: R12.1, U5-D.OUT
- removed net N$24: D1.K, D2.K, R23.1, U5-C.EN
- removed net N$25: R10.2, U5-D.IN
- removed net N$26: R11.2, U5-D.EN
- removed net N$27: R13.2, U3-B.+
- removed net N$28: R15.2, R16.1, U3-A.-
- removed net N$29: TP4.P$1, U3-B.OUT
- removed net N$8: KB_TRIM.2, KB_TRIM.3, R4.1
- removed net N$9: EXP_VCO_TRIM.2, EXP_VCO_TRIM.3, R5.1
- removed net PULSE: PULSE.P$1, R22.2, TYPE-SW.B, U3-A.OUT
- removed net PWM_CV: PWM_CV.1, R15.1
- removed net SAW: R24.2, TYPE-SW.A
- removed net VCO_CORE: R24.1, SAW.P$1, U3-A.+, U4-C.-, U4-C.OUT, U4-D.-
- removed net VCO_MOD_CV: R3.1, VCO_MOD_CV.1
- removed net VCO_OUT: CP_VCO_OUT.PAD, TYPE-SW.C, VCO_OUT.1
- new net C0: C.1, C2.1, E.1, G#.1, U16.Q0
- new net C1: A.1, C#.1, F.1, U16.Q1
- new net C2: A#.1, D.1, F#.1, U16.Q2
- new net C3: B.1, D#.1, G.1, U16.Q3
- new net D-BUS_CLK: U14E.Y, U15-CTL.CLK
- new net GATE: C48.1, GATE.1, U14D.Y
- new net KB_CLK: U1-A.Y, U16.EN, U18A.!CLK, U19.EN
- new net MR: C47.2, D7.K, R77.2, U18A.RST, U18B.RST
- new net N$102: C46.1, D5.A, R74.1, U14D.A
- new net N$103: R76.1, U15-CTL.!CLR
- new net N$104: U14B.Y, U14C.A
- new net N$105: U15-3.D, U18B.Q2, U19.A
- new net N$106: U15-4.D, U18B.Q3, U19.B
- new net N$107: C45.1, R75.1, U14A.A
- new net N$108: R75.2, U1-A.A, U14A.Y
- new net N$109: U15-1.D, U16.A, U18A.Q2
- new net N$110: U15-2.D, U16.B, U18A.Q3, U18B.EN
- new net N$111: R83.2, R84.2, R85.1
- new net N$112: C47.1, D5.K, U14E.A, U14F.Y
- new net N$113: R82.2, R85.2, R86.1
- new net N$114: D8.K, U14B.A
- new net N$115: C48.2, D8.A, R78.2
- new net N$116: C49.1, R79.2, U14F.A, U19.COM
- new net N$117: R81.2, R86.2, R87.1
- new net N$118: R80.2, R87.2, U13-A.+
- new net N$119: GLIDE.1, U13-A.-, U13-A.OUT
- new net N$120: C.2, D6.A
- new net N$121: C50.1, GLIDE.2, GLIDE.3, U13-B.+
- new net N$122: C#.2, D9.A
- new net N$123: D.2, D10.A
- new net N$124: D#.2, D11.A
- new net N$125: D12.A, E.2
- new net N$126: D13.A, F.2
- new net N$127: D14.A, F#.2
- new net N$128: D15.A, G.2
- new net N$129: D16.A, G#.2
- new net N$130: A.2, D17.A
- new net N$131: A#.2, D18.A
- new net N$132: B.2, D19.A
- new net N$133: C2.2, D20.A
- new net N$78: R57.1, U16.COM
- new net Q0: R83.1, U15-1.Q
- new net Q1: R82.1, U15-2.Q
- new net Q2: R81.1, U15-3.Q
- new net Q3: R80.1, U15-4.Q
- new net R0: D10.K, D11.K, D6.K, D9.K, U19.Q0
- new net R1: D12.K, D13.K, D14.K, D15.K, U19.Q1
- new net R2: D16.K, D17.K, D18.K, D19.K, U19.Q2
- new net R3: D20.K, U19.Q3
- new net TRIG: TRIG.1, U14C.Y
- net +5V: now also C43.1, C44.1, C51.1, C52.1, C59.1, PWR.3, R57.2, R74.2, R76.2, U1-PWR.VCC, U14PWR.VCC, U15-CTL.VCC, U16.VDD, U18-PWR.VCC, U18A.EN, U19.VDD; no longer C2.2, C5.1, J1.3, R16.2, R22.1, U5-A.IN
- net +9V: now also C53.1, PWR.1, U13-PWR.V+; no longer C10.2, C3.2, C6.2, C7.2, FREQ.3, J1.1, U3-PWR.V+, U4-PWR.V+, U5-B.OUT, U5-C.OUT, U5-PWR.VCC
- net -9V: now also C54.2, PWR.2, U13-PWR.V-; no longer C4.1, FREQ.1, J1.2, R8.1, U4-PWR.V-
- net GND: now also C43.2, C44.2, C45.2, C46.2, C49.2, C50.2, C51.2, C52.2, C53.2, C54.1, C59.2, D7.A, GATE.2, PWR.4, R77.1, R78.1, R79.1, R84.1, TRIG.2, U1-A.!EN, U1-PWR.GND, U14PWR.GND, U15-CTL.GND, U16.C, U16.VEE, U16.VSS, U18-PWR.GND, U18B.!CLK, U19.C, U19.VEE, U19.VSS; no longer BIAS.1, C2.1, C3.1, C4.2, C6.1, C7.1, C8.1, D2.A, J1.4, PWM_CV.2, Q1-A.COLLECTOR, Q1-B.BASE, R10.1, R11.1, R13.1, R14.1, R20.2, R23.2, R9.1, TYPE-MTG.MT1, TYPE-MTG.MT2, U3-PWR.V-, U4-A.+, U5-PWR.GND, VCO_MOD_CV.2, VCO_OUT.2
- net KB_CV: now also CP_KB_CV.PAD, U13-B.-, U13-B.OUT; no longer KB_TRIM.1
Other:
- note added: "===> EG"
- note added: "===> VCO"
- note added: "==> CV_PANEL"
- note added: "KEYBOARD"
- note removed: "=> VCF / CV_PNL"
- note removed: "Aquarius"
- note removed: "CP =>"
- note removed: "KB =>"
- note removed: "PULSE"
- note removed: "SAW"
- note removed: "VCO"
- note removed: "VCO FREQ"
- note removed: "VCO WAVE"
- note removed: "VCO_MOD =>"
- note removed: "Zodiac Synth"
- moved on the sheet: CP_GND, GLYPH, KB_CV, PCB

Commit message: Almost ready for FAB.
Sagittarius was mis-spelled, renamed it.  Taurus is still WIP.
Parts:
- removed C43: 0.1uF, rlc:CAPACITOR0603
- removed D17, D18, D19, D20: 1N4148, diodes:DIODE-1N4148
- added C.2: Tact. Sw., switch-smd:PUSHBTN-MOMB3FS
- added C5, C6: 1uF, rlc:CAPACITOR0603
- added D1, D2, D3, D4: 1N4148, diodes:DIODE-1N4148
- added VR: 5V, regulators:LDO-3P--5V-SOT23
- C2: value Tact. Sw. -> 0.1uF; device switch-smd:PUSHBTN-MOMB3FS -> rlc:CAPACITOR0603
- PWR: value (none) -> JST, 3P, VT, SMT; device con-jst:04P-VT-SMT -> con-jst:03P-VT-SMT
- renumbered C44 to C3, C45 to C1, C46 to C12, C47 to C13, C48 to C14, C49 to C11, C50 to C15, C51 to C7, C52 to C8, C53 to C9, C54 to C10, C59 to C4, GATE to GATE2EG, KB_CV to KB2VCO, R57 to R2, R74 to R5, R75 to R1, R76 to R3, R77 to R6, R78 to R7, R79 to R4, R80 to R8, R81 to R9, R82 to R10, R83 to R11, R84 to R15, R85 to R14, R86 to R13, R87 to R12, TRIG to TRIG2EG, U13 to U7, U14 to U6, U15 to U5, U16 to U3, U18 to U2, U19 to U4
Connections:
- net +5V: now also C2.1, C6.1, VR.VOUT; no longer C43.1, PWR.3
- net +9V: now also C5.1, VR.VIN
- net C0: now also C.2.1; no longer C2.1
- net GND: now also C2.2, C5.2, C6.2, D2.A, PWR.3, VR.GND; no longer C43.2, D7.A, PWR.4
- net MR: now also D2.K; no longer D7.K
- net N$102: now also D1.A; no longer D5.A
- net N$112: now also D1.K; no longer D5.K
- net N$114: now also D3.K; no longer D8.K
- net N$115: now also D3.A; no longer D8.A
- net N$120: now also D4.A; no longer D6.A
- net N$122: now also D5.A; no longer D9.A
- net N$123: now also D6.A; no longer D10.A
- net N$124: now also D7.A; no longer D11.A
- net N$125: now also D8.A; no longer D12.A
- net N$126: now also D9.A; no longer D13.A
- net N$127: now also D10.A; no longer D14.A
- net N$128: now also D11.A; no longer D15.A
- net N$129: now also D12.A; no longer D16.A
- net N$130: now also D13.A; no longer D17.A
- net N$131: now also D14.A; no longer D18.A
- net N$132: now also D15.A; no longer D19.A
- net N$133: now also C.2.2, D16.A; no longer C2.2, D20.A
- net R0: now also D4.K, D5.K, D7.K; no longer D10.K, D11.K, D9.K
- net R1: now also D10.K, D11.K, D8.K, D9.K; no longer D12.K, D13.K, D14.K, D15.K
- net R2: now also D12.K, D13.K, D14.K, D15.K; no longer D16.K, D17.K, D18.K, D19.K
- net R3: now also D16.K; no longer D20.K
Other:
- moved on the sheet: D10, D11, D12, D13, D14, D15, D16, D5, D6, D7, D8, D9
