File: PCB/synth-zodiac-cancer-led.brd (EAGLE design)
At the start: 76.1 x 72.4 mm, 50 parts, among them U1 ATmega328P-AU, X1 16MHz, X2 16MHz, X3 16MHz

Commit message: Perhaps final Rev. A?
Changed lines of the file:
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@@
 <attribute name="VALUE" x="48.5" y="15" size="0.4064" layer="28" rot="MR0" align="center"/>
 </element>
-<element name="C4" library="rlc" library_urn="urn:adsk.eagle:library:4192893" package="0603-CAP" package3d_urn="urn:adsk.eagle:package:4193021/4" value="18pF" x="49.4" y="22.1" smashed="yes" rot="MR270">
+<element name="C4" library="rlc" library_urn="urn:adsk.eagle:library:4192893" package="0603-CAP" package3d_urn="urn:adsk.eagle:package:4193021/5" value="18pF" x="49.4" y="22.1" smashed="yes" rot="MR270">
 <attribute name="COST01" value="0.12" x="49.4" y="22.1" size="1.778" layer="28" rot="MR270" display="off"/>
 <attribute name="COST10" value="0.09" x="49.4" y="22.1" size="1.778" layer="28" rot="MR270" display="off"/>
@@
 <attribute name="VALUE" x="49.4" y="22.1" size="0.2" layer="28" rot="MR270" align="center"/>
 </element>
-<element name="C5" library="rlc" library_urn="urn:adsk.eagle:library:4192893" package="0603-CAP" package3d_urn="urn:adsk.eagle:package:4193021/4" value="18pF" x="44" y="22.1" smashed="yes" rot="MR90">
+<element name="C5" library="rlc" library_urn="urn:adsk.eagle:library:4192893" package="0603-CAP" package3d_urn="urn:adsk.eagle:package:4193021/5" value="18pF" x="44" y="22.1" smashed="yes" rot="MR90">
 <attribute name="COST01" value="0.12" x="44" y="22.1" size="1.778" layer="28" rot="MR90" display="off"/>
 <attribute name="COST10" value="0.09" x="44" y="22.1" size="1.778" layer="28" rot="MR90" display="off"/>
@@
 <attribute name="VALUE" x="49.646" y="37.3" size="0.2" layer="28" rot="MR90" align="center"/>
 </element>
-<element name="C1" library="rlc" library_urn="urn:adsk.eagle:library:4192893" package="0603-CAP" package3d_urn="urn:adsk.eagle:package:4193021/4" value="0.1uF" x="47.2" y="37.3" smashed="yes" rot="MR90">
+<element name="C1" library="rlc" library_urn="urn:adsk.eagle:library:4192893" package="0603-CAP" package3d_urn="urn:adsk.eagle:package:4193021/5" value="0.1uF" x="47.2" y="37.3" smashed="yes" rot="MR90">
 <attribute name="COST01" value="0.12" x="47.2" y="37.3" size="1.778" layer="28" rot="MR90" display="off"/>
 <attribute name="COST10" value="0.09" x="47.2" y="37.3" size="1.778" layer="28" rot="MR90" display="off"/>
@@
 <attribute name="VALUE" x="36.4" y="15.5" size="0.3" layer="28" font="vector" rot="MR0" align="center"/>
 </element>
-<element name="C6" library="rlc" library_urn="urn:adsk.eagle:library:4192893" package="0603-CAP" package3d_urn="urn:adsk.eagle:package:4193021/4" value="1uF" x="34.1" y="15.5" smashed="yes" rot="MR90">
+<element name="C6" library="rlc" library_urn="urn:adsk.eagle:library:4192893" package="0603-CAP" package3d_urn="urn:adsk.eagle:package:4193021/5" value="1uF" x="34.1" y="15.5" smashed="yes" rot="MR90">
 <attribute name="COST01" value="0.12" x="34.1" y="15.5" size="1.778" layer="28" rot="MR90" display="off"/>
 <attribute name="COST10" value="0.09" x="34.1" y="15.5" size="1.778" layer="28" rot="MR90" display="off"/>
@@
 <attribute name="VALUE" x="34.1" y="15.5" size="0.2" layer="28" rot="MR90" align="center"/>
 </element>
-<element name="C7" library="rlc" library_urn="urn:adsk.eagle:library:4192893" package="0603-CAP" package3d_urn="urn:adsk.eagle:package:4193021/4" value="1uF" x="38.8" y="15.5" smashed="yes" rot="MR270">
+<element name="C7" library="rlc" library_urn="urn:adsk.eagle:library:4192893" package="0603-CAP" package3d_urn="urn:adsk.eagle:package:4193021/5" value="1uF" x="38.8" y="15.5" smashed="yes" rot="MR270">
 <attribute name="COST01" value="0.12" x="38.8" y="15.5" size="1.778" layer="28" rot="MR270" display="off"/>
 <attribute name="COST10" value="0.09" x="38.8" y="15.5" size="1.778" layer="28" rot="MR270" display="off"/>
@@
 <attribute name="VALUE" x="49.2" y="29.7" size="0.6096" layer="28" font="vector" rot="MR90" align="center"/>
 </element>
-<element name="C3" library="rlc" library_urn="urn:adsk.eagle:library:4192893" package="0603-CAP" package3d_urn="urn:adsk.eagle:package:4193021/4" value="0.1uF" x="51.7" y="22.1" smashed="yes" rot="MR270">
+<element name="C3" library="rlc" library_urn="urn:adsk.eagle:library:4192893" package="0603-CAP" package3d_urn="urn:adsk.eagle:package:4193021/5" value="0.1uF" x="51.7" y="22.1" smashed="yes" rot="MR270">
 <attribute name="COST01" value="0.12" x="51.7" y="22.1" size="1.778" layer="28" rot="MR270" display="off"/>
 <attribute name="COST10" value="0.09" x="51.7" y="22.1" size="1.778" layer="28" rot="MR270" display="off"/>
@@
 <attribute name="VALUE" x="65.472075" y="39.66095" size="0.4064" layer="28" font="vector" rot="MR108" align="center"/>
 </element>
-<element name="DEC" library="switch-smd" library_urn="urn:adsk.eagle:library:5542824" package="B3FS-BACKMOUNT" package3d_urn="urn:adsk.eagle:package:41392463/3" value="SPST, TACT, MOM" x="32" y="49.5" smashed="yes" rot="R270">
+<element name="DEC" library="switch-smd" library_urn="urn:adsk.eagle:library:5542824" package="B3FS-BACKMOUNT" package3d_urn="urn:adsk.eagle:package:41392463/4" value="SPST, TACT, MOM" x="32" y="49.5" smashed="yes" rot="R270">
 <attribute name="COST01" value="0.15" x="32" y="49.5" size="1.778" layer="27" rot="R270" display="off"/>
 <attribute name="COST10" value="0.12" x="32" y="49.5" size="1.778" layer="27" rot="R270" display="off"/>
@@
 <attribute name="MFR" value="CK" x="32" y="49.5" size="1.778" layer="27" rot="R270" display="off"/>
 <attribute name="MPN" value="B3FS" x="32" y="49.5" size="1.778" layer="27" rot="R270" display="off"/>
-<attribute name="MPN2" value="Tayda A-3961(2.3mm), A-3959(1.4mm), A-3962" x="32" y="49.5" size="1.778" layer="27" rot="R270" display="off"/>
+<attribute name="MPN2" value="Tayda A-3961(2.3mm), A-5134(3.14mm,RA)" x="32" y="49.5" size="1.778" layer="27" rot="R270" display="off"/>
+<attribute name="NAME" x="31.8" y="48.5" size="0.7" layer="25" font="vector" ratio="15" rot="SR0" align="center"/>
 <attribute name="NAME" x="32.053" y="44.883" size="0.7" layer="26" font="vector" ratio="15" rot="SMR0" align="center"/>
-<attribute name="NAME" x="31.8" y="48.5" size="0.7" layer="25" font="vector" ratio="15" rot="SR0" align="center"/>
 <attribute name="VALUE" x="29.189" y="49.5" size="0.3" layer="27" font="vector" rot="R270" align="center"/>
 </element>
@@
 <attribute name="VALUE" x="46.6" y="17.9" size="0.4064" layer="28" ratio="15" rot="MR0" align="top-center"/>
 </element>
-<element name="C2" library="rlc" library_urn="urn:adsk.eagle:library:4192893" package="0603-CAP" package3d_urn="urn:adsk.eagle:package:4193021/4" value="0.1uF" x="51.1" y="37.3" smashed="yes" rot="MR270">
+<element name="C2" library="rlc" library_urn="urn:adsk.eagle:library:4192893" package="0603-CAP" package3d_urn="urn:adsk.eagle:package:4193021/5" value="0.1uF" x="51.1" y="37.3" smashed="yes" rot="MR270">
 <attribute name="COST01" value="0.12" x="51.1" y="37.3" size="1.778" layer="28" rot="MR270" display="off"/>
 <attribute name="COST10" value="0.09" x="51.1" y="37.3" size="1.778" layer="28" rot="MR270" display="off"/>
@@
 <attribute name="VALUE" x="43.946" y="37.3" size="0.2" layer="28" rot="MR90" align="center"/>
 </element>
-<element name="INC" library="switch-smd" library_urn="urn:adsk.eagle:library:5542824" package="B3FS-BACKMOUNT" package3d_urn="urn:adsk.eagle:package:41392463/3" value="SPST, TACT, MOM" x="44" y="49.5" smashed="yes" rot="R270">
+<element name="INC" library="switch-smd" library_urn="urn:adsk.eagle:library:5542824" package="B3FS-BACKMOUNT" package3d_urn="urn:adsk.eagle:package:41392463/4" value="SPST, TACT, MOM" x="44" y="49.5" smashed="yes" rot="R270">
 <attribute name="COST01" value="0.15" x="42.2" y="48.5" size="1.778" layer="27" rot="R270" display="off"/>
 <attribute name="COST10" value="0.12" x="42.2" y="48.5" size="1.778" layer="27" rot="R270" display="off"/>
@@
 <attribute name="MFR" value="CK" x="42.2" y="48.5" size="1.778" layer="27" rot="R270" display="off"/>
 <attribute name="MPN" value="B3FS" x="42.2" y="48.5" size="1.778" layer="27" rot="R270" display="off"/>
-<attribute name="MPN2" value="Tayda A-3961(2.3mm), A-3959(1.4mm), A-3962" x="42.2" y="48.5" size="1.778" layer="27" rot="R270" display="off"/>
+<attribute name="MPN2" value="Tayda A-3961(2.3mm), A-5134(3.14mm,RA)" x="42.2" y="48.5" size="1.778" layer="27" rot="R270" display="off"/>
+<attribute name="NAME" x="44.2" y="48.6" size="0.7" layer="25" font="vector" ratio="15" rot="SR0" align="center"/>
 <attribute name="NAME" x="43.953" y="45.083" size="0.7" layer="26" font="vector" ratio="15" rot="SMR0" align="center"/>
-<attribute name="NAME" x="44.2" y="48.6" size="0.7" layer="25" font="vector" ratio="15" rot="SR0" align="center"/>
 <attribute name="VALUE" x="41.189" y="49.5" size="0.3" layer="27" font="vector" rot="R270" align="center"/>
 </element>
