File: PCB/synth-zodiac-cancer-led.sch (EAGLE design)
At the start: 67 parts, among them Q1 NPN, Q2 NPN, U1 TL071, U3 ATmega328P-AU, X1 16MHz, X2 16MHz, X3 16MHz

Commit message: Work in progress for rev A,  VCO rev.B
Parts:
- removed A0, A1, A2, A3, A4, A5, A6, A7, RX, TX: PADSMD-050X050, con-testpoints:PADSMD-050X050
- removed C10, C11: 18pF, rlc:CAPACITOR0603
- removed C12, C15, C16, C17, C9: 0.1uF, rlc:CAPACITOR0603
- removed C13, C14: 1uF, rlc:CAPACITOR0603
- removed C8: 0.47uF, rlc:CAPACITOR0603
- removed COW: SPST, TACT, MOM, switch-smd:PUSHBTN-MOMB3FS-BLIND
- removed COW2VCA: JST, SH, 2P, con-jst:02P-SM-VT-SMT
- removed D1, D2, D3: 1N4148, diodes:DIODE-1N4148
- removed ENV: TPSMD-040-RND, con-testpoints:TPSMD-040-RND
- removed ICSP: Connector, 6P, SM, VT, con-jst:06P-SM-VT-SMT
- removed Q1, Q2: NPN, transistor-bjt:NPN-BC846
- removed R10, R13: 33K, rlc:RESISTOR0603
- removed R11: 470K, rlc:RESISTOR0603
- removed R12, R14: 100, rlc:RESISTOR0603
- removed R7: 10K, rlc:RESISTOR0603
- removed R8: 100K, rlc:RESISTOR0603
- removed R9: 2.2K, rlc:RESISTOR0603
- removed U3: ATmega328P-AU, atmel-atmega:ATMEGA328AU
- removed VR: 5V, regulators:LDO-3P--5V-SOT23
- added ADC6, ADC7, PD0, PD1, PD4: PADSMD-050X050, con-testpoints:PADSMD-050X050
- added DEC, INC: SPST, TACT, MOM, switch-smd:PUSHBTN-MOMB3FS-BLIND
- added IN0, IN1, IN2, IN3, IN4, IN5, V3.7: JST, SH, 2P, con-jst:02P-SM-VT-SMT
- added ISCP: Connector, 6P, SM, VT, con-jst:06P-SM-VT-SMT
- added RGB1: SK2812B_3535, led:SMART_LED3535
- added RGB2, RGB3, RGB4, RGB5: (no value), led:SMART_LED4020-SIDE
- added RGBX: 3P, Male, Breakaway, 2.54mm, con-headers:CON_03X1-2.54MM-SMT-EDGE
- added VR1: 5V, regulators:LDO-3P--5V-SOT23
- C1, C3: value 10uF/16V -> 0.1uF
- C2: value 0.0022uF -> 0.1uF
- C4: value 0.0022uF -> 18pF
- C5: value 0.0033uF -> 18pF
- C6: value 0.01uF -> 1uF
- CONST1: device circuit-monkey-zodiac:CONSTELLATION-TAURUS -> circuit-monkey-zodiac:CONSTELLATION-CANCER
- GLYPH1: device circuit-monkey-zodiac:GLYPH-TAURUS -> circuit-monkey-zodiac:GLYPH-CANCER
- R1: value 470K -> 10K
- R2: value 470K -> 470
- R3: value 100 -> 470
- R4: value 10K -> 4.7K
- R5: value 100K -> 10K
- R6: value 100 -> 330
- U1: value TL071 -> ATmega328P-AU; device op-amp:SINGLE-TL071 -> atmel-atmega:ATMEGA328AU
- X1: device xtal:2PCTS_445 -> xtal:2P3.2X2.5
- X2: device xtal:RESONATOR-CSTE16 -> xtal:2PCTS_445
- X3: device xtal:2P3.2X2.5 -> xtal:RESONATOR-CSTE16
Connections:
- removed net COW: C5.2, R11.2, R12.1, U1G.OUT
- removed net COW_OUT: COW2VCA.1, R12.2
- removed net ENV: C8.1, D3.K, ENV.P$1, R10.1, R5.2, R8.2
- removed net MIX: C2.2, C4.2, C5.1, C6.1, R9.2
- removed net N$10: C4.1, R7.2
- removed net N$13: C6.2, R11.1, U1G.-
- removed net N$15: C7.1, R10.2
- removed net N$19: A0.PAD, U3.PC0
- removed net N$20: A1.PAD, U3.PC1
- removed net N$21: A2.PAD, U3.PC2
- removed net N$22: A3.PAD, U3.PC3
- removed net N$23: A4.PAD, U3.PC4
- removed net N$24: A5.PAD, U3.PC5
- removed net PULSE_1MS: D3.A, U3.PD7
- removed net SQ_540: C3.1, U3.PD5
- removed net SQ_800: C1.1, U3.PD6
- new net +4.1V: RGB1.VDD, RGB2.VDD, RGB3.VDD, RGB4.VDD, RGB5.VDD, RGBX.2, V3.7.1
- new net AIN0: IN0.1, U1.PC0
- new net AIN1: IN1.1, U1.PC1
- new net AIN2: IN2.1, U1.PC2
- new net AIN3: IN3.1, U1.PC3
- new net AIN4: IN4.1, U1.PC4
- new net AIN5: IN5.1, U1.PC5
- new net BTN_2: R2.1, U1.PD6
- new net LED: R4.1, U1.PD5
- net !RST: now also C2.1, ISCP.5, R1.2, U1.PC6; no longer C17.1, ICSP.5, R13.2, U3.PC6
- net +5V: now also C1.1, C3.1, C7.1, ISCP.2, R1.1, U1.AVCC, U1.VCC@4, U1.VCC@6, VR1.VOUT; no longer C12.1, C14.1, C15.1, ICSP.2, R13.1, U3.AVCC, U3.VCC@4, U3.VCC@6, VR.VOUT
- net +9V: now also C6.1, VR1.VIN; no longer C13.1, C9.1, R1.2, R2.2, U1PWR.V+, VR.VIN
- net -9V: no longer C16.2, U1PWR.V-
- net BTN_1: now also R3.1, U1.PD7; no longer R14.1, U3.PD4
- net GND: now also C1.2, C2.2, C3.2, C4.2, C5.2, C6.2, DEC.2, IN0.2, IN1.2, IN2.2, IN3.2, IN4.2, IN5.2, INC.2, ISCP.6, R5.1, RGB1.GND, RGB2.GND, RGB3.GND, RGB4.GND, RGB5.GND, RGBX.3, U1.AGND, U1.GND@3, U1.GND@5, V3.7.2, VR1.GND, X3.2; no longer C10.2, C11.2, C12.2, C13.2, C14.2, C15.2, C16.1, C17.2, C8.2, C9.2, COW.2, COW2VCA.2, ICSP.6, R3.1, R6.1, R9.1, U1G.+, U3.AGND, U3.GND@3, U3.GND@5, VR.GND, X2.2
- net MISO: now also ISCP.1, U1.PB4; no longer ICSP.1, U3.PB4
- net MOSI: now also ISCP.4, U1.PB3; no longer ICSP.4, U3.PB3
- net N$1: now also INC.1, R3.2; no longer D1.K, Q1.COLLECTOR
- net N$11: now also DEC.1, R2.2; no longer COW.1, R14.2
- net N$12: now also U1.PD3; no longer U3.PD3
- net N$14: now also U1.PD2; no longer U3.PD2
- net N$16: now also U1.PB2; no longer U3.PB2
- net N$17: now also U1.PB1; no longer U3.PB1
- net N$18: now also U1.PB0; no longer U3.PB0
- net N$2: now also RGB1.OUT, RGB2.IN; no longer Q1.EMITTER, R3.2
- net N$25: now also ADC6.PAD, U1.ADC6; no longer A6.PAD, U3.ADC6
- net N$26: now also ADC7.PAD, U1.ADC7; no longer A7.PAD, U3.ADC7
- net N$27: now also U1.AREF; no longer U3.AREF
- net N$3: now also RGB2.OUT, RGB3.IN; no longer C1.2, Q1.BASE, R1.1
- net N$4: now also RGB3.OUT, RGB4.IN; no longer D1.A, R4.1, R5.1
- net N$5: now also RGB4.OUT, RGB5.IN; no longer C2.1, R4.2
- net N$6: now also R6.2, RGBX.1; no longer D2.K, Q2.COLLECTOR
- net N$7: now also R4.2, R5.2, RGB1.IN; no longer Q2.EMITTER, R6.2
- net N$8: now also PD4.PAD, U1.PD4; no longer C3.2, Q2.BASE, R2.1
- net N$9: now also R6.1, RGB5.OUT; no longer D2.A, R7.1, R8.1
- net RX: now also PD0.PAD, U1.PD0; no longer RX.PAD, U3.PD0
- net SCK: now also ISCP.3, U1.PB5; no longer ICSP.3, U3.PB5
- net TX: now also PD1.PAD, U1.PD1; no longer TX.PAD, U3.PD1
- net XTAL1: now also C4.1, U1.PB6, X2.P$1, X3.1; no longer C10.1, U3.PB6, X2.1, X3.P$1
- net XTAL2: now also C5.1, U1.PB7, X2.P$2, X3.3; no longer C11.1, U3.PB7, X2.3, X3.P$2
Other:
- note added: "Cancer"
- note added: "LED FX"
- note removed: "=> VCA"
- note removed: "Cowbell"
- note removed: "ENV"
- note removed: "Pulse 1mS"
- note removed: "Sq. 540Hz"
- note removed: "Sq. 800Hz"
- note removed: "Taurus"
- moved on the sheet: AREF, C1, C2, C3, C4, C5, C6, C7, CONST1, GLYPH1, GND, PB0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
