File: PCB/synth-zodiac-sagittarius-speaker.brd (EAGLE design)
At the start: 76.1 x 72.4 mm, 14 parts

Commit message: Work in progress for rev A,  VCO rev.B
Parts:
- removed PWR-3.7V: 2-pin, VT, SMT, con-jst:B2B-PH-SM4
- added PWR-3.7: JST, SH, 2P, con-jst:BM02B-SRSS-TB
- VCA_IN: value 2-pin, VT, SMT -> JST, SH, 2P; device con-jst:B2B-PH-SM4 -> con-jst:BM02B-SRSS-TB
- moved VCA_IN 13.8 mm to (52.8, 47.0), turned to 90 degrees
Connections:
- net GND: now also PWR-3.7.2; no longer PWR-3.7V.2
- net VDD: now also PWR-3.7.1; no longer PWR-3.7V.1
Routing:
- net N$3: track 35.2 -> 7.80 mm
- net VDD: track 25.2 -> 22.4 mm

Commit message: Perhaps final Rev. A?
Other:
- board text added: "CUT OUT"
Changed lines of the file:
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@@
 <text x="19.3" y="51.5" size="1" layer="1" ratio="20" rot="R36" align="top-center">S A T A N ' S    C Y C L E    W O R K S</text>
 <text x="19.3" y="51.5" size="1" layer="29" ratio="20" rot="R36" align="top-center">S A T A N ' S    C Y C L E    W O R K S</text>
+<text x="38" y="28.8" size="3" layer="20" align="center">CUT OUT</text>
 </plain>
 <attributes>
@@
 <elements>
 <element name="PCB1" library="circuit-monkey-zodiac" library_urn="urn:adsk.eagle:library:36060312" package="PENTAGON-40MM-RAD" package3d_urn="urn:adsk.eagle:package:36376820/2" value="PCB FAB" x="38" y="33" smashed="yes"/>
-<element name="VOL" library="rlc" library_urn="urn:adsk.eagle:library:4192893" package="POT-RV9110" package3d_urn="urn:adsk.eagle:package:36472483/2" value="10K" x="38" y="55" smashed="yes" rot="MR306">
+<element name="VOL" library="rlc" library_urn="urn:adsk.eagle:library:4192893" package="POT-RV9110" package3d_urn="urn:adsk.eagle:package:36472483/3" value="10K" x="38" y="55" smashed="yes" rot="MR306">
 <attribute name="COST01" value="0.70" x="38" y="55" size="1.778" layer="28" rot="MR306" display="off"/>
 <attribute name="COST10" value="0.60" x="38" y="55" size="1.778" layer="28" rot="MR306" display="off"/>
@@
 <attribute name="VALUE" x="17.8" y="46.1" size="0.3" layer="28" rot="MR270" align="center"/>
 </element>
-<element name="C1" library="rlc" library_urn="urn:adsk.eagle:library:4192893" package="0603-CAP" package3d_urn="urn:adsk.eagle:package:4193021/4" value="0.1uF" x="22.8" y="45.9" smashed="yes" rot="MR0">
+<element name="C1" library="rlc" library_urn="urn:adsk.eagle:library:4192893" package="0603-CAP" package3d_urn="urn:adsk.eagle:package:4193021/5" value="0.1uF" x="22.8" y="45.9" smashed="yes" rot="MR0">
 <attribute name="COST01" value="0.12" x="22.8" y="45.9" size="1.778" layer="28" rot="MR0" display="off"/>
 <attribute name="COST10" value="0.09" x="22.8" y="45.9" size="1.778" layer="28" rot="MR0" display="off"/>
@@
 <attribute name="VALUE" x="22.8" y="45.9" size="0.2" layer="28" rot="MR0" align="center"/>
 </element>
-<element name="C2" library="rlc" library_urn="urn:adsk.eagle:library:4192893" package="0603-CAP" package3d_urn="urn:adsk.eagle:package:4193021/4" value="0.1uF" x="22.8" y="43.3" smashed="yes" rot="MR0">
+<element name="C2" library="rlc" library_urn="urn:adsk.eagle:library:4192893" package="0603-CAP" package3d_urn="urn:adsk.eagle:package:4193021/5" value="0.1uF" x="22.8" y="43.3" smashed="yes" rot="MR0">
 <attribute name="COST01" value="0.12" x="22.8" y="43.3" size="1.778" layer="28" rot="MR0" display="off"/>
 <attribute name="COST10" value="0.09" x="22.8" y="43.3" size="1.778" layer="28" rot="MR0" display="off"/>
@@
 <attribute name="VALUE" x="22.8" y="46.946" size="0.2" layer="28" rot="MR0" align="center"/>
 </element>
-<element name="C3" library="rlc" library_urn="urn:adsk.eagle:library:4192893" package="0603-CAP" package3d_urn="urn:adsk.eagle:package:4193021/4" value="4.7uF" x="22.8" y="48.5" smashed="yes" rot="MR0">
+<element name="C3" library="rlc" library_urn="urn:adsk.eagle:library:4192893" package="0603-CAP" package3d_urn="urn:adsk.eagle:package:4193021/5" value="4.7uF" x="22.8" y="48.5" smashed="yes" rot="MR0">
 <attribute name="COST01" value="0.12" x="22.8" y="48.5" size="1.778" layer="28" rot="MR0" display="off"/>
 <attribute name="COST10" value="0.09" x="22.8" y="48.5" size="1.778" layer="28" rot="MR0" display="off"/>
@@
 <attribute name="VALUE" x="22.8" y="44.346" size="0.2" layer="28" rot="MR0" align="center"/>
 </element>
-<element name="C4" library="rlc" library_urn="urn:adsk.eagle:library:4192893" package="0603-CAP" package3d_urn="urn:adsk.eagle:package:4193021/4" value="10uF" x="12.5" y="42.6" smashed="yes" rot="MR90">
+<element name="C4" library="rlc" library_urn="urn:adsk.eagle:library:4192893" package="0603-CAP" package3d_urn="urn:adsk.eagle:package:4193021/5" value="10uF" x="12.5" y="42.6" smashed="yes" rot="MR90">
 <attribute name="COST01" value="0.12" x="12.5" y="42.6" size="1.778" layer="28" rot="MR90" display="off"/>
 <attribute name="COST10" value="0.09" x="12.5" y="42.6" size="1.778" layer="28" rot="MR90" display="off"/>
@@
 <attribute name="VALUE" x="12.5" y="42.6" size="0.2" layer="28" rot="MR90" align="center"/>
 </element>
-<element name="C5" library="rlc" library_urn="urn:adsk.eagle:library:4192893" package="0603-CAP" package3d_urn="urn:adsk.eagle:package:4193021/4" value="1uF" x="13.8" y="42.6" smashed="yes" rot="MR90">
+<element name="C5" library="rlc" library_urn="urn:adsk.eagle:library:4192893" package="0603-CAP" package3d_urn="urn:adsk.eagle:package:4193021/5" value="1uF" x="13.8" y="42.6" smashed="yes" rot="MR90">
 <attribute name="COST01" value="0.12" x="13.8" y="42.6" size="1.778" layer="28" rot="MR90" display="off"/>
 <attribute name="COST10" value="0.09" x="13.8" y="42.6" size="1.778" layer="28" rot="MR90" display="off"/>
