File: PCB/synth-zodiac-sagittarius-speaker.sch (EAGLE design)
At the start: 14 parts

Commit message: Work in progress for rev A,  VCO rev.B
Parts:
- removed PWR-3.7V: 2-pin, VT, SMT, con-jst:02PVT-SMT
- added PWR-3.7: JST, SH, 2P, con-jst:02P-SM-VT-SMT
- VCA_IN: value 2-pin, VT, SMT -> JST, SH, 2P; device con-jst:02PVT-SMT -> con-jst:02P-SM-VT-SMT
Connections:
- net GND: now also PWR-3.7.2; no longer PWR-3.7V.2
- net VDD: now also PWR-3.7.1; no longer PWR-3.7V.1
Other:
- note added: "Amp & Speaker"
- note added: "SATAN'S CYCLE WORKS"
- note added: "Sagittarius"
- note added: "Zodiac Synth"
- moved on the sheet: AMP, C1, C2, C3, C4, C5, R1, R2, R3, SPKR, VCA_IN, VOL
