File: PCB/synth-zodiac-scorpio-kbd-mcu.brd (EAGLE design)
At the start: 76.1 x 72.4 mm, 58 parts, among them U1 ATmega328P-MU, U2 TL072A, X1 16MHz

Commit message: Tune values and some schematic visual tweaks.
Parts:
- R16: value 10.0M -> 10K
